File: nas.brd (EAGLE design)
At the start: 100 x 80 mm, 93 parts, among them J1 RASPBERRYPI-40-PIN-GPIO_PTH_N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, U1 RASPBERRY_PI_CM-1-1376408-4, U2 SPX29302, U3 SPX29302, U4 SPX29302, U5 SPX29302, U6 SPX29302, U7 TLV1117-33CDCY, Y1 12MHz, Y2 12MHz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

Commit message: Breaking up into many pages
Parts:
- added C48, C49: 10pf, SparkFun-Capacitors:1206
- added C50, C51, C52, C53: 10n, SparkFun-Capacitors:1206
- added R23: 12k, SparkFun-Resistors:1206
- added R24: 22, SparkFun-Resistors:1206
- added R25: 1M, SparkFun-Resistors:1206
- added R26: 1.2K, SparkFun-Resistors:1206
- added SH2: SHORT-HT5, shorts-old:SHORT_TOP-50
- added U$16: PL-2571-B, SparkFun:SSOP28DB
- added U$17: SATA_POWER_AND_DATA, geusebio:3M-SATA-5622-1200-ML
- added Y5: 30Mhz, SparkFun-Clocks:CRYSTAL-SMD-5X3.2-4PAD
- moved U$15 527.7 mm to (115.0, 30.0)
- moved C39 521.9 mm to (147.0, 35.5), turned to 270 degrees
- moved C38 520.4 mm to (150.0, 35.5), turned to 270 degrees
- moved C37 518.8 mm to (153.0, 35.5), turned to 270 degrees
- moved C36 517.3 mm to (156.0, 35.5), turned to 270 degrees
- moved U$12 475.6 mm to (150.0, 44.0), turned to 180 degrees
- moved J1 364.4 mm to (-38.7, 39.7), turned to 90 degrees
- moved U1 89.6 mm to (-49.5, 72.4)
- moved U2 61.6 mm to (-49.5, 19.1)
- renumbered U$5 to USB_A, U$7 to USB_B, U$9 to USB_C
Connections:
- removed net USB_B1_M: U$12.4, USB_B.10
- removed net USB_B1_P: U$12.3, USB_B.11
- new net N$30: R23.2, U$16.1
- new net N$33: C49.2, R25.1, U$16.7, Y5.1
- new net N$34: R24.2, R25.2, U$16.6
- new net N$35: C48.2, R24.1, Y5.3
- new net N$36: R26.1, U$16.20
- new net SATA_2_AGND: C48.1, C49.1, R26.2, SH2.2, U$16.16, U$16.21, U$16.25
- new net SATA_2_CON_RXDN: C52.2, U$17.P$5
- new net SATA_2_CON_RXDP: C53.2, U$17.P$6
- new net SATA_2_CON_TXDN: C51.2, U$17.P$3
- new net SATA_2_CON_TXDP: C50.2, U$17.P$2
- new net SATA_2_IC_RXDN: C52.1, U$16.24
- new net SATA_2_IC_RXDP: C53.1, U$16.23
- new net SATA_2_IC_TXDN: C51.1, U$16.26
- new net SATA_2_IC_TXDP: C50.1, U$16.27
- new net SATA_2_VCC1.2D: U$16.19, U$16.28, U$16.8, U$16.9
- new net SATA_2_VCC3.3D: U$16.13, U$16.17, U$16.22, U$16.5
- net 12V: now also U$17.P$20, U$17.P$21, U$17.P$22
- net 5V: now also U$16.18
- net GND: now also R23.1, SH2.1, U$16.2, U$17.P$1, U$17.P$11, U$17.P$12, U$17.P$13, U$17.P$17, U$17.P$19, U$17.P$4, U$17.P$7
- net SATA_A_3.3V: now also U$17.P$10, U$17.P$8, U$17.P$9
- net SATA_A_5V: now also U$17.P$14, U$17.P$15, U$17.P$16
- net USB_B2_M: now also U$12.4, U$16.4, USB_B.10
- net USB_B2_P: now also U$12.3, U$16.3, USB_B.11
- net USB_VBUS: now also U$16.10
Routing:
- net SATA_2_CON_RXDP: track 0.00 -> 7.75 mm
- net SATA_2_IC_RXDP: track 0.00 -> 7.42 mm
- net SATA_2_CON_TXDP: track 0.00 -> 6.63 mm
- net SATA_2_CON_RXDN: track 0.00 -> 6.01 mm
- net SATA_2_IC_TXDP: track 0.00 -> 5.87 mm
- net SATA_2_CON_TXDN: track 0.00 -> 5.56 mm
- net SATA_2_IC_RXDN: track 0.00 -> 5.07 mm
- net SATA_2_IC_TXDN: track 0.00 -> 3.52 mm
Other:
- board size 100 x 80 mm -> 100 x 160 mm
