File: nas.sch (EAGLE design)
At the start: 93 parts, among them J1 RASPBERRYPI-40-PIN-GPIO_PTH_N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, U1 RASPBERRY_PI_CM-1-1376408-4, U2 SPX29302, U3 SPX29302, U4 SPX29302, U5 SPX29302, U6 SPX29302, U7 TLV1117-33CDCY, Y1 12MHz, Y2 12MHz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

Commit message: Breaking up into many pages
Parts:
- removed U$5, U$7, U$9: FE1.1S, imcom:FE1.1S
- added C48, C49: 10pf, SparkFun-Capacitors:10UF-1206-6.3V-20%
- added C50, C51, C52, C53: 10n, SparkFun-Capacitors:10UF-1206-6.3V-20%
- added R23: 12k, SparkFun-Resistors:RESISTOR1206
- added R24: 22, SparkFun-Resistors:RESISTOR1206
- added R25: 1M, SparkFun-Resistors:RESISTOR1206
- added R26: 1.2K, SparkFun-Resistors:RESISTOR1206
- added SH2: SHORT-HT5, shorts-old:SHORT-HT5
- added U$16: PL-2571-B, SparkFun:SSOP28
- added U$17: SATA_POWER_AND_DATA, geusebio:SATA_POWER_AND_DATA
- added USB_A, USB_B, USB_C: FE1.1S, imcom:FE1.1S
- added Y5: 30Mhz, SparkFun-Clocks:CRYSTAL-12MHZ"
Connections:
- removed net USB_B1_M: U$12.4, U$7.DM1
- removed net USB_B1_P: U$12.3, U$7.DP1
- new net N$30: R23.2, U$16.1
- new net N$33: C49.2, R25.1, U$16.7, Y5.1
- new net N$34: R24.2, R25.2, U$16.6
- new net N$35: C48.2, R24.1, Y5.2
- new net N$36: R26.1, U$16.20
- new net SATA_2_AGND: C48.1, C49.1, R26.2, SH2.P$2, U$16.16, U$16.21, U$16.25
- new net SATA_2_CON_RXDN: C52.2, U$17.RECEIVE-
- new net SATA_2_CON_RXDP: C53.2, U$17.RECEIVE+
- new net SATA_2_CON_TXDN: C51.2, U$17.TRANSMIT-
- new net SATA_2_CON_TXDP: C50.2, U$17.TRANSMIT+
- new net SATA_2_IC_RXDN: C52.1, U$16.24
- new net SATA_2_IC_RXDP: C53.1, U$16.23
- new net SATA_2_IC_TXDN: C51.1, U$16.26
- new net SATA_2_IC_TXDP: C50.1, U$16.27
- new net SATA_2_VCC1.2D: U$16.19, U$16.28, U$16.8, U$16.9
- new net SATA_2_VCC3.3D: U$16.13, U$16.17, U$16.22, U$16.5
- net 12V: now also U$17.12V
- net 5V: now also U$16.18, USB_A.VDD5, USB_B.VDD5, USB_C.VDD5; no longer U$5.VDD5, U$7.VDD5, U$9.VDD5
- net GND: now also R23.1, SH2.P$1, U$16.2, U$17.D_GND, U$17.P_GND, USB_A.VSS, USB_B.VSS, USB_C.VSS; no longer U$5.VSS, U$7.VSS, U$9.VSS
- net HOST_USB_DM_N: now also USB_A.DMU; no longer U$5.DMU
- net HOST_USB_DP_P: now also USB_A.DPU; no longer U$5.DPU
- net N$10: now also USB_B.BUSJ, USB_B.OVCJ, USB_B.VBUSM, USB_B.VD33, USB_B.VD33_O, USB_B.XRSTJ; no longer U$7.BUSJ, U$7.OVCJ, U$7.VBUSM, U$7.VD33, U$7.VD33_O, U$7.XRSTJ
- net N$11: now also USB_A.REXT; no longer U$5.REXT
- net N$12: now also USB_B.REXT; no longer U$7.REXT
- net N$13: now also USB_C.XIN; no longer U$9.XIN
- net N$14: now also USB_C.DM4; no longer U$9.DM4
- net N$15: now also USB_C.DP4; no longer U$9.DP4
- net N$16: now also USB_C.DM3; no longer U$9.DM3
- net N$17: now also USB_C.DP3; no longer U$9.DP3
- net N$18: now also USB_C.DM2; no longer U$9.DM2
- net N$19: now also USB_C.DP2; no longer U$9.DP2
- net N$20: now also USB_C.DM1; no longer U$9.DM1
- net N$21: now also USB_C.DP1; no longer U$9.DP1
- net N$23: now also USB_C.XOUT; no longer U$9.XOUT
- net N$24: now also USB_C.VD18, USB_C.VD18_O; no longer U$9.VD18, U$9.VD18_O
- net N$25: now also USB_C.BUSJ, USB_C.OVCJ, USB_C.VBUSM, USB_C.VD33, USB_C.VD33_O, USB_C.XRSTJ; no longer U$9.BUSJ, U$9.OVCJ, U$9.VBUSM, U$9.VD33, U$9.VD33_O, U$9.XRSTJ
- net N$26: now also USB_C.REXT; no longer U$9.REXT
- net N$3: now also USB_A.VD18, USB_A.VD18_O; no longer U$5.VD18, U$5.VD18_O
- net N$4: now also USB_A.BUSJ, USB_A.OVCJ, USB_A.VBUSM, USB_A.VD33, USB_A.VD33_O, USB_A.XRSTJ; no longer U$5.BUSJ, U$5.OVCJ, U$5.VBUSM, U$5.VD33, U$5.VD33_O, U$5.XRSTJ
- net N$5: now also USB_B.XIN; no longer U$7.XIN
- net N$6: now also USB_A.XIN; no longer U$5.XIN
- net N$7: now also USB_A.XOUT; no longer U$5.XOUT
- net N$8: now also USB_B.XOUT; no longer U$7.XOUT
- net N$9: now also USB_B.VD18, USB_B.VD18_O; no longer U$7.VD18, U$7.VD18_O
- net SATA_A_3.3V: now also U$17.3.3V
- net SATA_A_5V: now also U$17.5V
- net USB_A1_M: now also USB_A.DM1, USB_B.DMU; no longer U$5.DM1, U$7.DMU
- net USB_A1_P: now also USB_A.DP1, USB_B.DPU; no longer U$5.DP1, U$7.DPU
- net USB_A2_M: now also USB_A.DM2, USB_C.DMU; no longer U$5.DM2, U$9.DMU
- net USB_A2_P: now also USB_A.DP2, USB_C.DPU; no longer U$5.DP2, U$9.DPU
- net USB_A3_M: now also USB_A.DM3; no longer U$5.DM3
- net USB_A3_P: now also USB_A.DP3; no longer U$5.DP3
- net USB_A4_M: now also USB_A.DM4; no longer U$5.DM4
- net USB_A4_P: now also USB_A.DP4; no longer U$5.DP4
- net USB_B2_M: now also U$12.4, U$16.4, USB_B.DM1, USB_B.DM2; no longer U$7.DM2
- net USB_B2_P: now also U$12.3, U$16.3, USB_B.DP1, USB_B.DP2; no longer U$7.DP2
- net USB_B3_M: now also USB_B.DM3; no longer U$7.DM3
- net USB_B3_P: now also USB_B.DP3; no longer U$7.DP3
- net USB_B4_M: now also USB_B.DM4; no longer U$7.DM4
- net USB_B4_P: now also USB_B.DP4; no longer U$7.DP4
- net USB_VBUS: now also U$16.10
